File: pcb/fiberboard-logic.kicad_sch (KiCad schematic)
At the start: 59 parts, among them J1 VIN, J3 FOOT, J4 NPN, J5 RLY1, J6 RLY2, J7 SOL, J8 RS485, J9 OLED, K1 G6KU-2F-Y, K2 G6KU-2F-Y, Q12 AO4407A, Q3 2N3904, Q4 2N3904, Q5 AO3400A, U1 ESP32-DevKitC, U2 XL1509-5.0, U3 AMS1117-3.3, U5 PC817, U6 PC817, U7 MAX485E

Commit message: thêm các linh kiện bảo vệ nguồn và sửa layout để lắp vào hộp PLC 45x90x40mm 2 hàng giắc
Parts:
- removed J9: OLED, Connector_PinHeader_2.54mm:PinHeader_1x04_P2.54mm_Horizontal, symbol Fiberboard:Screw_Terminal_01x04
- added C19: 10uF, Capacitor_SMD:C_0805_2012Metric, symbol Device:C
- added C21, C23, C25: 100nF, Capacitor_SMD:C_0805_2012Metric, symbol Device:C
- added C22, C24: 220uF, Capacitor_SMD:CP_Elec_6.3x5.4, symbol Device:C
- added D10, D11, D12, D9: SMAJ5.0A, Diode_SMD:D_SMA, symbol Device:D_TVS
- added F2: 5x20 F0.5A, Fiberboard:Fuseholder_5x20mm_Horizontal, symbol Device:Fuse
- added F3: 5x20 F0.25A, Fiberboard:Fuseholder_5x20mm_Horizontal, symbol Device:Fuse
- added FB1, FB2, FB3, FB4: BLM21PG121, Inductor_SMD:L_0805_2012Metric, symbol Device:L
- added J2: KB24, Fiberboard:Terminal_2EDG5.08-1x02_P5.08mm_Horizontal, symbol Fiberboard:Screw_Terminal_01x02
- added L2: ACM2012, Inductor_SMD:L_CommonModeChoke_Coilank_ACM2012, symbol Fiberboard:CM_Choke_4
- added R18, R19: 10R, Resistor_SMD:R_0805_2012Metric, symbol Device:R
- added R20, R21: 100k, Resistor_SMD:R_0805_2012Metric, symbol Device:R
- added RV1: MOV-26V, Varistor:Varistor_Panasonic_VF, symbol Device:R
- C2: value 100uF -> 220uF; footprint Capacitor_SMD:C_1206_3216Metric -> Capacitor_SMD:CP_Elec_6.3x5.4
- C4: value 470uF -> 1000uF; footprint Capacitor_SMD:CP_Elec_10x10.5 -> Capacitor_SMD:CP_Elec_10x12.5
- D3, D4: value 1N4148 -> SS34
- D5: footprint Diode_SMD:D_SMA -> Diode_SMD:D_SOD-123
- F1: value MF-MSMF350 -> 5x20 F4A; footprint Fuse:Fuse_2920_7451Metric -> Fiberboard:Fuseholder_5x20mm_Horizontal
- J1, J3, J7: footprint TerminalBlock_Phoenix:TerminalBlock_Phoenix_MKDS-1,5-2-5.08_1x02_P5.08mm_Horizontal -> Fiberboard:Terminal_2EDG5.08-1x02_P5.08mm_Horizontal
- J4, J5, J6: footprint TerminalBlock_Phoenix:TerminalBlock_Phoenix_MKDS-1,5-3-5.08_1x03_P5.08mm_Horizontal -> Fiberboard:Terminal_2EDG5.08-1x03_P5.08mm_Horizontal
- J8: value RS485 -> RS485-2EDG3P; footprint TerminalBlock_Phoenix:TerminalBlock_Phoenix_MKDS-1,5-3-5.08_1x03_P5.08mm_Horizontal -> Fiberboard:Terminal_2EDG5.08-1x03_P5.08mm_Horizontal
- R13: value 100R -> 100
- R15: value 120R -> 100
- U1: value ESP32-DevKitC -> ESP32-DevKitC-32E
Connections:
- net +24V: now also F3.1, J2.1 (P1); no longer D5.1 (K), J7.1 (P1)
- net +3V3: now also C21.1, FB1.2; no longer C18.1, C3.1, U3.2 (VO)
- net +5V: now also C22.1, FB2.2, FB4.1; no longer C2.1, C5.1, D3.1 (K), D4.1 (K), K1.1 (COIL+), K2.1 (COIL+), L1.2
- net GND: now also U1.14 (GND), C21.2, C22.2, D10.2 (A2), D9.2 (A2), FB3.2, R20.2, R21.2; no longer NT1.2 (GND), U1.13 (GND), U6.2 (K)
- net GND_PWR: now also U6.2 (K), C19.2, C23.1, C24.2, C25.2, D11.1 (A1), D12.2 (A2), J2.2 (P2), L2.4, RV1.2; no longer J1.2 (P2)
- net IN_FOOT: now also R20.1
- net IN_NPN: now also R21.1
- net RS485_A: now also R18.1; no longer J8.1 (P1), R15.1
- net RS485_B: now also R19.1; no longer J8.2 (P2), R15.2
- net VIN_FUSE: now also C19.1, L2.2, RV1.1; no longer F1.2
- new net +24V_SOL: D5.1 (K), F3.2, J7.1 (P1)
- new net +3V3_REG: C18.1, C3.1, FB1.1, U3.2 (VO)
- new net +5V_RAW: C2.1, C5.1, FB2.1, L1.2
- new net +5V_RLY: C24.1, C25.1, D12.1 (A1), D3.1 (K), D4.1 (K), F2.1, F2.2, FB4.2, K1.1 (COIL+), K2.1 (COIL+)
- new net GND_SPLICE: C23.2, D11.2 (A2), FB3.1, NT1.2 (GND)
- new net RS485_A_BUS: D9.1 (A1), J8.1 (P1), R15.1, R18.2
- new net RS485_B_BUS: D10.1 (A1), J8.2 (P2), R15.2, R19.2
- new net VIN_CM_IN: F1.2, L2.1
- new net VIN_CM_RET: J1.2 (P2), L2.3
Other:
- note added: "J1->F1->L2->RV1/D7->Q12->C4 1mF | U2 XL1509 buck | C2/C22 5V bulk | U3 3.3V"
- note removed: "J1->F1->D7->Q12->C4 | U2 XL1509 buck 24V->5V | U3 AMS1117 5V->3.3V"

Commit message: chia vùng linh kiện để sắp xếp và tránh linh kiện quá dày
Parts:
- removed F2: 5x20 F0.5A, Fiberboard:Fuseholder_5x20mm_Horizontal, symbol Device:Fuse
- removed F3: 5x20 F0.25A, Fiberboard:Fuseholder_5x20mm_Horizontal, symbol Device:Fuse
- added C26: C 220uF, Capacitor_SMD:CP_Elec_6.3x5.4, symbol Device:C
- added C27: C 100nF, Capacitor_SMD:C_0805_2012Metric, symbol Device:C
- added D13: VIN, LED_SMD:LED_0805_2012Metric, symbol Device:LED
- added D14: KB24, LED_SMD:LED_0805_2012Metric, symbol Device:LED
- added D15: FOOT, LED_SMD:LED_0805_2012Metric, symbol Device:LED
- added D16: NPN, LED_SMD:LED_0805_2012Metric, symbol Device:LED
- added D17: RLY1, LED_SMD:LED_0805_2012Metric, symbol Device:LED
- added D18: RLY2, LED_SMD:LED_0805_2012Metric, symbol Device:LED
- added D19: VAN, LED_SMD:LED_0805_2012Metric, symbol Device:LED
- added D20: 485, LED_SMD:LED_0805_2012Metric, symbol Device:LED
- added D21: TX1, LED_SMD:LED_0805_2012Metric, symbol Device:LED
- added D22: RX1, LED_SMD:LED_0805_2012Metric, symbol Device:LED
- added D23: TX2, LED_SMD:LED_0805_2012Metric, symbol Device:LED
- added D24: RX2, LED_SMD:LED_0805_2012Metric, symbol Device:LED
- added D25: 5V, LED_SMD:LED_0805_2012Metric, symbol Device:LED
- added D26: SMAJ5.0A, Diode_SMD:D_SMA, symbol Device:D_TVS
- added D27: 24V, LED_SMD:LED_0805_2012Metric, symbol Device:LED
- added FB5: BLM21PG121, Inductor_SMD:L_0805_2012Metric, symbol Device:L
- added R22, R23, R28, R39: R 10k, Resistor_SMD:R_0805_2012Metric, symbol Device:R
- added R24, R25, R26, R27, R29, R30, R31, R32, R33, R34, R40, R41, R42, R43, R44, R45: R 1k, Resistor_SMD:R_0805_2012Metric, symbol Device:R
- C12, C13, C14, C15, C17, C18, C21, C23, C25, C5: value 100nF -> C 100nF
- C16, C19, C7: value 10uF -> C 10uF
- C2, C22, C24: value 220uF -> C 220uF
- C3: value 22uF -> C 22uF
- C4: value 1000uF -> C 1000uF
- D6: value STATUS -> 3V3
- R10, R14, R38, R9: value 10k -> R 10k
- R11, R12, R16, R37, R7, R8: value 1k -> R 1k
- R13, R15: value 100 -> R 100
- R17, R20, R21: value 100k -> R 100k
- R18, R19: value 10R -> R 10R
- R36: value 3k -> R 3k
Connections:
- net +24V_SOL is gone; now on net +24V: D5.1 (K), J7.1 (P1)
- net +24V: now also R38.1, U2.5 (GND), U2.6 (GND), U2.7 (GND), U2.8 (GND), R23.1, R28.1, R39.1
- net +3V3: now also R24.1, R25.1
- net +5V: now also FB5.1
- net +5V_RAW: now also R34.1
- net FIBER1_DIG: now also R42.2; no longer F1R.1 (DATA_OUT)
- net FIBER1_PWM: now also R30.1, R40.1; no longer F1T.4 (DATA_IN)
- net FIBER2_DIG: now also R43.2; no longer F2R.1 (DATA_OUT)
- net FIBER2_PWM: now also R32.1, R41.1; no longer F2T.4 (DATA_IN)
- net GND: now also D20.1 (K), D21.1 (K), D22.1 (K), D23.1 (K), D24.1 (K), D25.1 (K)
- net GND_PWR: now also C26.2, C27.2, D14.1 (K), D26.2 (A2), D27.1 (K); no longer R38.1, U2.5 (GND), U2.6 (GND), U2.7 (GND), U2.8 (GND)
- net IN_FOOT: now also D15.1 (K)
- net IN_NPN: now also D16.1 (K)
- net RLY1_COIL: now also D17.1 (K)
- net RLY2_COIL: now also D18.1 (K)
- net RS485_DE: now also R29.1
- net RS485_RX: now also R45.2; no longer U7.1 (RO)
- net RS485_TX: now also R44.1; no longer U7.4 (DI)
- net SOL_LO: now also D19.1 (K)
- net VIN_CM_RET: now also D13.1 (K)
- net VIN_RAW: now also R22.1
- net +5V_RLY renamed +5V_RLY1
- net +5V_RLY1: now also R26.1; no longer D4.1 (K), K2.1 (COIL+)
- net FOOT_LED renamed FOOT_AN
- net NPN_LED renamed NPN_AN
- net STAT_LED renamed P3V3_AN
- new net +5V_RLY2: C26.1, C27.1, D26.1 (A1), D4.1 (K), FB5.2, K2.1 (COIL+), R27.1
- new net F1R_AN: D22.2 (A), R31.2
- new net F1T_AN: D21.2 (A), R30.2
- new net F2R_AN: D24.2 (A), R33.2
- new net F2T_AN: D23.2 (A), R32.2
- new net FIBER1_RX: F1R.1 (DATA_OUT), R31.1, R42.1
- new net FIBER1_TX: F1T.4 (DATA_IN), R40.2
- new net FIBER2_RX: F2R.1 (DATA_OUT), R33.1, R43.1
- new net FIBER2_TX: F2T.4 (DATA_IN), R41.2
- new net J1_AN: D13.2 (A), R22.2
- new net J2_AN: D14.2 (A), R23.2
- new net J3_AN: D15.2 (A), R24.2
- new net J4_AN: D16.2 (A), R25.2
- new net J5_AN: D17.2 (A), R26.2
- new net J6_AN: D18.2 (A), R27.2
- new net J7_AN: D19.2 (A), R28.2
- new net J8_AN: D20.2 (A), R29.2
- new net P24_AN: D27.2 (A), R39.2
- new net P5V_AN: D25.2 (A), R34.2
- new net RS485_DI: R44.2, U7.4 (DI)
- new net RS485_RO: R45.1, U7.1 (RO)
Other:
- note added: "J1->F1->L2->RV1/D7->Q12->C4 | buck 5V | LDO 3.3V"
- note removed: "ESP32"
- note removed: "J1->F1->L2->RV1/D7->Q12->C4 1mF | U2 XL1509 buck | C2/C22 5V bulk | U3 3.3V"

Commit message: update lại linh kiện để tối ưu thương mại. chuyển sang dùng cảm biến sợi quang rời, không tích hợp trên mạch nữa
Parts:
- removed C12, C13, C21, C23, C25, C27: C 100nF, Capacitor_SMD:C_0805_2012Metric, symbol Device:C
- removed C19: C 10uF, Capacitor_SMD:C_0805_2012Metric, symbol Device:C
- removed C22, C24, C26: C 220uF, Capacitor_SMD:CP_Elec_6.3x5.4, symbol Device:C
- removed D10, D11, D12, D26, D9: SMAJ5.0A, Diode_SMD:D_SMA, symbol Device:D_TVS
- removed D13: VIN, LED_SMD:LED_0805_2012Metric, symbol Device:LED
- removed D14: KB24, LED_SMD:LED_0805_2012Metric, symbol Device:LED
- removed D21: TX1, LED_SMD:LED_0805_2012Metric, symbol Device:LED
- removed D22: RX1, LED_SMD:LED_0805_2012Metric, symbol Device:LED
- removed D23: TX2, LED_SMD:LED_0805_2012Metric, symbol Device:LED
- removed D24: RX2, LED_SMD:LED_0805_2012Metric, symbol Device:LED
- removed D25: 5V, LED_SMD:LED_0805_2012Metric, symbol Device:LED
- removed D5, D8: SS34, Diode_SMD:D_SOD-123, symbol Device:D
- removed F1R, F2R: AFBR-2624Z, Fiberboard:AFBR_2624Z_VL, symbol Fiberboard:AFBR_2624Z
- removed F1T, F2T: AFBR-1624Z, Fiberboard:AFBR_1624Z_VL, symbol Fiberboard:AFBR_1624Z
- removed FB1, FB2, FB3, FB4, FB5: BLM21PG121, Inductor_SMD:L_0805_2012Metric, symbol Device:L
- removed K1, K2: G6KU-2F-Y, Fiberboard:G6KU-2F_SMD, symbol Fiberboard:G5LE-1
- removed L2: ACM2012, Inductor_SMD:L_CommonModeChoke_Coilank_ACM2012, symbol Fiberboard:CM_Choke_4
- removed Q12: AO4407A, Package_TO_SOT_SMD:SOT-23, symbol Transistor_FET:Q_PMOS_GSD
- removed Q3, Q4: 2N3904, Package_TO_SOT_SMD:SOT-23, symbol Transistor_BJT:2N3904
- removed R20, R21: R 100k, Resistor_SMD:R_0805_2012Metric, symbol Device:R
- removed R22, R23, R38: R 10k, Resistor_SMD:R_0805_2012Metric, symbol Device:R
- removed R30, R31, R32, R33, R34, R37, R40, R41, R42, R43, R44, R45: R 1k, Resistor_SMD:R_0805_2012Metric, symbol Device:R
- removed R36: R 3k, Resistor_SMD:R_0805_2012Metric, symbol Device:R
- removed RV1: MOV-26V, Varistor:Varistor_Panasonic_VF, symbol Device:R
- removed U1: ESP32-DevKitC-32E, Fiberboard:ESP32_DevKitC_Socket, symbol Fiberboard:ESP32_DevKitC_Socket
- removed U7: MAX485E, Package_SO:SOIC-8_3.9x4.9mm_P1.27mm, symbol Interface_UART:MAX485E
- added C10: C 1uF, Capacitor_SMD:C_0805_2012Metric, symbol Device:C
- added C11, C9: C 100nF, Capacitor_SMD:C_0805_2012Metric, symbol Device:C
- added C8: C 10uF, Capacitor_SMD:C_0805_2012Metric, symbol Device:C
- added D30: RUN, LED_SMD:LED_0805_2012Metric, symbol Device:LED
- added D31: AMP1, LED_SMD:LED_0805_2012Metric, symbol Device:LED
- added D32: AMP2, LED_SMD:LED_0805_2012Metric, symbol Device:LED
- added D5, D8: SS34, Diode_SMD:D_SMA, symbol Device:D_Schottky
- added D9: PSM712, Package_TO_SOT_SMD:SOT-23, symbol Diode:SM712_SOT23
- added J10: AMP2, Fiberboard:Terminal_2EDG5.08-1x03_P5.08mm_Horizontal, symbol Fiberboard:Screw_Terminal_01x03
- added J11: USB-C, Connector_USB:USB_C_Receptacle_HRO_TYPE-C-31-M-12, symbol Connector:USB_C_Receptacle_USB2.0_16P
- added J9: AMP1, Fiberboard:Terminal_2EDG5.08-1x03_P5.08mm_Horizontal, symbol Fiberboard:Screw_Terminal_01x03
- added K1, K2: HF3FF-024-1ZS, Relay_THT:Relay_SPDT_SANYOU_SRD_Series_Form_C, symbol Relay:SANYOU_SRD_Form_C
- added Q12: AO3401A, Package_TO_SOT_SMD:SOT-23, symbol Transistor_FET:AO3401A
- added Q3, Q4: MMBT3904, Package_TO_SOT_SMD:SOT-23, symbol Transistor_BJT:MMBT3904
- added R47, R48, R49, R52, R53, R54, R55, R57, R58, R60, R61, R63: R 10k, Resistor_SMD:R_0805_2012Metric, symbol Device:R
- added R50, R51: R 5.1k, Resistor_SMD:R_0805_2012Metric, symbol Device:R
- added R56, R59, R62: R 1k, Resistor_SMD:R_0805_2012Metric, symbol Device:R
- added SW1: BOOT, Button_Switch_SMD:SW_Push_1P1T_XKB_TS-1187A, symbol Switch:SW_Push
- added U1: ESP32-C3-WROOM-02, RF_Module:ESP32-C3-WROOM-02, symbol RF_Module:ESP32-C3-WROOM-02
- added U10, U9: LTV-817S, Package_DIP:SMDIP-4_W9.53mm, symbol Fiberboard:PC817
- added U7: SP3485EN, Package_SO:SOIC-8_3.9x4.9mm_P1.27mm, symbol Interface_UART:MAX3485
- C14, C15, C17: value C 100nF -> C 100nF 50V; LCSC (none) -> C49678
- C16: value C 10uF -> C 10uF 50V; footprint Capacitor_SMD:C_0805_2012Metric -> Capacitor_SMD:C_1206_3216Metric; LCSC (none) -> C13585
- C18, C5: LCSC (none) -> C49678
- C2: value C 220uF -> C 220uF 10V; LCSC (none) -> C2833309
- C3: LCSC (none) -> C45783
- C4: value C 1000uF -> C 470uF 35V; footprint Capacitor_SMD:CP_Elec_10x12.5 -> Capacitor_SMD:CP_Elec_10x10.5; LCSC (none) -> C2836436
- C7: LCSC (none) -> C15850
- D15, D16, D17, D18, D19, D20, D27, D6: LCSC (none) -> C84256
- D3, D4: value SS34 -> 1N4148W; LCSC (none) -> C81598
- D7: value SMAJ28A -> SMAJ26A; LCSC (none) -> C2848697
- F1: value 5x20 F4A -> 5x20 su 4A; footprint Fiberboard:Fuseholder_5x20mm_Horizontal -> Fiberboard:Fuseholder_5x20mm_Covered
- J8: value RS485-2EDG3P -> RS485
- L1: value 47uH -> 47uH 6045; footprint Inductor_SMD:L_1210_3225Metric -> Inductor_SMD:L_Sunlord_SWPA6045S; LCSC (none) -> C36414
- Q5: LCSC (none) -> C20917
- R10, R14, R28, R39, R9: LCSC (none) -> C17414
- R11, R12, R16, R24, R25, R29: LCSC (none) -> C17513
- R13: value R 100 -> R 10R; LCSC (none) -> C17415
- R15: value R 100 -> R 120R; LCSC (none) -> C17437
- R17: value R 100k -> R 27k; LCSC (none) -> C17593
- R18, R19: LCSC (none) -> C17415
- R26, R27, R7, R8: value R 1k -> R 10k; LCSC (none) -> C17414
- U2: footprint Package_TO_SOT_SMD:TO-263-5_TabPin3 -> Package_SO:SOIC-8_3.9x4.9mm_P1.27mm; LCSC (none) -> C61063
- U3: LCSC (none) -> C6186
- U5, U6: value PC817 -> LTV-817S; footprint Fiberboard:PC817_SO4 -> Package_DIP:SMDIP-4_W9.53mm; LCSC (none) -> C109227
Connections:
- net +3V3_REG is gone; now on net +3V3: C18.1, C3.1, U3.2 (VO)
- net +5V_RAW is gone; now on net +5V: C2.1, C5.1, L1.2
- net +5V_RLY1 is gone; now on net +24V: D3.1 (K), R26.1
- net +5V_RLY2 is gone; now on net +24V: D4.1 (K), R27.1
- net BUCK_EN is gone; now on net GND_PWR: U2.4 (~{EN})
- net BUCK_FB is gone; now on net +5V: U2.3 (FB)
- net GND_SPLICE is gone; now on net GND: NT1.2 (GND)
- net NPN_V+ is gone; now on net +24V: J4.1 (P1)
- net VIN_CM_IN is gone; now on net VIN_FUSE: F1.2
- net VIN_CM_RET is gone; now on net GND_PWR: J1.2 (P2)
- net +24V: now also R7.1, R8.1, D5.1 (K), J10.1 (P1), J9.1 (P1), K1.5, K2.5, Q12.2 (S), R57.1, R60.1, R63.1; no longer U2.5 (GND), U2.6 (GND), U2.7 (GND), U2.8 (GND)
- net +3V3: now also C11.1, C8.1, C9.1, R52.1, R53.1, R54.1, R55.1, R56.1, R58.1, R59.1, R61.1, R62.1, U1.1 (3V3), U7.8 (VCC)
- net FET_G: now also Q12.1 (G), R63.2
- net GND: now also C10.2, C11.2, C8.2, C9.2, D9.3 (common), J11.A1 (GND), J11.A12 (GND), J11.B1 (GND), J11.B12 (GND), J11.SH (SHIELD), R49.2, R50.2, R51.2, SW1.2, U1.19 (GND), U1.9 (GND), U10.3 (E), U7.5 (GND), U9.3 (E); no longer C2.2, C5.2
- net GND_PWR: now also C2.2, C5.2, J3.2 (P2), U2.5 (GND), U2.6 (GND), U2.7 (GND), U2.8 (GND), D8.2 (A), J10.3 (P3), J9.3 (P3), Q3.2 (E), Q4.2 (E), R47.2, R48.2; no longer U6.2 (K)
- net IN_FOOT: now also U1.3 (IO4)
- net IN_NPN: now also U1.4 (IO5)
- net NPN_SIG: now also U6.2 (K); no longer R8.1
- net OUT_MOS: now also U1.10 (IO10)
- net OUT_RLY1: now also U1.18 (IO0)
- net OUT_RLY2: now also U1.17 (IO1)
- net RLY1_B: now also Q3.1 (B), R47.1
- net RLY1_COIL: now also K1.2, Q3.3 (C)
- net RLY1_COM: now also K1.1
- net RLY1_NC: now also K1.4
- net RLY1_NO: now also K1.3
- net RLY2_B: now also Q4.1 (B), R48.1
- net RLY2_COIL: now also K2.2, Q4.3 (C)
- net RLY2_COM: now also K2.1
- net RLY2_NC: now also K2.4
- net RLY2_NO: now also K2.3
- net RS485_A: now also U7.6 (A)
- net RS485_A_BUS: now also D9.1 (A1)
- net RS485_B: now also U7.7 (B)
- net RS485_B_BUS: now also D9.2 (A2)
- net RS485_DE: now also R49.1, U1.15 (IO3), U7.2 (~{RE}), U7.3 (DE)
- net RS485_RX: now also U1.11 (IO20/RXD), U7.1 (RO)
- net RS485_TX: now also U1.12 (IO21/TXD), U7.4 (DI)
- net SOL_LO: now also D5.2 (A)
- net VIN_FUSE: now also Q12.3 (D)
- net +5V_SW renamed BUCK_SW
- net BUCK_SW: now also D8.1 (K)
- net FOOT_A renamed FOOT_SIG
- net FOOT_SIG: now also U5.2 (K); no longer R7.1
- removed net FOOT_K: J3.2 (P2), U5.2 (K)
- new net: J11.A4 (VBUS), J11.A9 (VBUS), J11.B4 (VBUS), J11.B9 (VBUS)
- new net AMP1_AN: R57.2, U9.1 (A)
- new net AMP1_SIG: J9.2 (P2), U9.2 (K)
- new net AMP2_AN: R60.2, U10.1 (A)
- new net AMP2_SIG: J10.2 (P2), U10.2 (K)
- new net ESP_BOOT: R55.2, SW1.1, U1.8 (IO9)
- new net ESP_EN: C10.1, R52.2, U1.2 (EN)
- new net ESP_IO2: R53.2, U1.16 (IO2)
- new net IN_AMP1: D31.1 (K), R58.2, U1.5 (IO6), U9.4 (C)
- new net IN_AMP2: D32.1 (K), R61.2, U1.6 (IO7), U10.4 (C)
- new net J10_AN: D32.2 (A), R62.2
- new net J9_AN: D31.2 (A), R59.2
- new net LED_RUN: D30.1 (K), R54.2, U1.7 (IO8)
- new net RUN_AN: D30.2 (A), R56.2
- new net USB_CC1: J11.A5 (CC1), R50.1
- new net USB_CC2: J11.B5 (CC2), R51.1
- new net USB_DN: J11.A7 (D-), J11.B7 (D-), U1.13 (IO18)
- new net USB_DP: J11.A6 (D+), J11.B6 (D+), U1.14 (IO19)
- no-connect marks 18 -> 6
Other:
- note added: "4 ISOLATED NPN INPUTS (PC817): FOOT / NPN / AMP1 / AMP2"
- note added: "FIBERBOARD AIO — FULLY NET-CONNECTED SCHEMATIC (rev B)"
- note added: "MCU ESP32-C3-WROOM-02 + USB-C (USBLC6)"
- note added: "POWER: J1->F1->D7 TVS->Q12 P-FET (reverse) -> +24V | XL1509-3.3 buck"
- note added: "RELAYS 24V COIL / SOLENOID MOSFET / RS485 3V3"
- note removed: "DIGITAL IN"
- note removed: "FIBER CH1"
- note removed: "FIBER CH2"
- note removed: "FIBERBOARD AIO — FULLY NET-CONNECTED SCHEMATIC (rev A3)"
- note removed: "J1->F1->L2->RV1/D7->Q12->C4 | buck 5V | LDO 3.3V"
- note removed: "POWER / 24V IN PROTECT"
- note removed: "RELAYS / MOSFET / RS485"
